Commit message: feat: added camera

File: Project2/catkin_ws/src/my_robot/urdf/my_robot.xacro (robot description, xacro)
@@ -70,6 +70,5 @@
           ixx="0.1" ixy="0" ixz="0"
           iyy="0.1" iyz="0"
-          izz="0.1"
-      />
+          izz="0.1" />
     </inertial>
     <collision name='left_wheel_collision'>
@@ -101,6 +100,5 @@
           ixx="0.1" ixy="0" ixz="0"
           iyy="0.1" iyz="0"
-          izz="0.1"
-      />
+          izz="0.1" />
     </inertial>
     <collision name='right_wheel_collision'>
@@ -117,3 +115,32 @@
     </visual>
   </link>
+  <joint type="fixed" name="camera_joint">
+    <axis   xyz="0.0 1 0" rpy="0.0 0 0"/>
+    <origin xyz="0.2 0 0" rpy="0.0 0 0"/>
+    <parent link="chassis"/>
+    <child  link='camera' />
+  </joint>
+  <link name='camera'>
+    <inertial>
+      <mass value="0.1"/>
+      <origin xyz=" 0.0 0 0" rpy="0.0 0 0"/>
+      <box_inertia m="0.1" x="0.05" y="0.05" z="0.05"/>
+      <inertia
+          ixx="1e-6" ixy="0" ixz="0"
+          iyy="1e-6" iyz="0"
+          izz="1e-6" />
+    </inertial>
+    <visual name='camera_visual'>
+      <origin xyz=" 0.0 0 0" rpy="0.0 0 0"/>
+      <geometry>
+        <box size="0.05 0.05 0.05"/>
+      </geometry>
+    </visual>
+    <collision name='camera_collision'>
+      <origin xyz=" 0.0 0 0" rpy="0.0 0 0"/>
+      <geometry>
+        <box size="0.05 0.05 0.05"/>
+      </geometry>
+    </collision>
+  </link>
 </robot>

Commit message: feat: Porject2 - 7 tested

File: Project2/catkin_ws/src/my_robot/urdf/my_robot.xacro (robot description, xacro)
@@ -144,3 +144,43 @@
     </collision>
   </link>
+  <joint type="fixed" name="hokuyo_joint">
+    <axis   xyz="0.0 1 0" rpy="0.0 0 0"/>
+    <origin xyz="0.15 0 .1" rpy="0.0 0 0"/>
+    <parent link="chassis"/>
+    <child  link='hokuyo' />
+  </joint>
+  <link name='hokuyo'>
+    <inertial>
+      <mass value="1e-5"/>
+      <origin xyz="0.0 0 0" rpy="0.0 0 0"/>
+      <inertia
+          ixx="1e-6" ixy="0" ixz="0"
+          iyy="1e-6" iyz="0"
+          izz="1e-6" />
+    </inertial>
+    <visual name="hokuyo_visual">
+      <origin xyz="0.0 0 0" rpy="0.0 0 0"/>
+      <geometry>
+        <mesh filename="package://my_robot/meshes/hokuyo.dae" />
+      </geometry>
+    </visual>
+    <inertial name="hokuyo_inertial">
+      <origin xyz="0.0 0 0" rpy="0.0 0 0"/>
+      <geometry>
+        <box size= "0.1 0.1 0.1"/>
+      </geometry>
+    </inertial>
+  </link>
+  <gazebo reference="left_wheel">
+    <material>Gazebo/Black</material>
+  </gazebo>
+  <gazebo reference="right_wheel">
+    <material>Gazebo/Black</material>
+  </gazebo>
+  <gazebo reference="chassis">
+    <material>Gazebo/Blue</material>
+  </gazebo>
+  <gazebo reference="camera">
+    <material>Gazebo/Black</material>
+  </gazebo>
 </robot>
